File: schematic/macro9000.kicad_sch (KiCad schematic)
At the start: 19 parts, among them SW1 SW_Push, SW2 SW_Push, SW3 SW_Push, SW4 SW_Push, SW5 SW_Push, SW6 SW_Push, SW7 SW_Push, SW8 SW_Push, SW9 SW_Push

Commit message: added firmware + updated readme for that
Parts:
- added J1: AudioPlug4, symbol Connector_Audio:AudioPlug4
Connections:
- net at RZ1.21 (3V3): now also J1.S
- net at RZ1.22 (GND): now also J1.T
- net at RZ1.7 (GP6): now also J1.R2
- net at RZ1.8 (GP7): now also J1.R1
Other:
- moved on the sheet: RZ1
Changed lines of the file:
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@@
+	(wire
+		(pts
+			(xy 158.75 76.2) (xy 158.75 68.58)
+		)
+		(stroke
+			(width 0)
+			(type default)
+		)
+	)
 	(wire
 		(pts
@@
 	(wire
 		(pts
+			(xy 132.08 57.15) (xy 132.08 31.75)
+		)
+		(stroke
+			(width 0)
+			(type default)
+		)
+	)
+	(wire
+		(pts
+			(xy 138.43 59.69) (xy 138.43 55.88)
+		)
+		(stroke
+			(width 0)
+			(type default)
+		)
+	)
+	(wire
+		(pts
 			(xy 60.96 58.42) (xy 73.66 58.42)
 		)
@@
 	(wire
 		(pts
+			(xy 132.08 31.75) (xy 160.02 31.75)
+		)
+		(stroke
+			(width 0)
+			(type default)
+		)
+	)
+	(wire
+		(pts
 			(xy 73.66 71.12) (xy 88.9 71.12)
 		)
@@
 	(wire
 		(pts
+			(xy 132.08 76.2) (xy 158.75 76.2)
+		)
+		(stroke
+			(width 0)
+			(type default)
+		)
+	)
+	(wire
+		(pts
+			(xy 132.08 59.69) (xy 138.43 59.69)
+		)
+		(stroke
+			(width 0)
+			(type default)
+		)
+	)
+	(wire
+		(pts
+			(xy 132.08 64.77) (xy 132.08 76.2)
+		)
+		(stroke
+			(width 0)
+			(type default)
+		)
+	)
+	(wire
+		(pts
 			(xy 63.5 38.1) (xy 63.5 50.8)
 		)
@@
 	(wire
 		(pts
+			(xy 142.24 58.42) (xy 144.78 58.42)
+		)
+		(stroke
+			(width 0)
+			(type default)
+		)
+	)
+	(wire
+		(pts
 			(xy 48.26 45.72) (xy 60.96 45.72)
 		)
@@
 	(wire
 		(pts
+			(xy 142.24 62.23) (xy 142.24 58.42)
+		)
+		(stroke
+			(width 0)
+			(type default)
+		)
+	)
+	(wire
+		(pts
 			(xy 63.5 50.8) (xy 63.5 63.5)
 		)
@@
 	(wire
 		(pts
+			(xy 132.08 62.23) (xy 142.24 62.23)
+		)
+		(stroke
+			(width 0)
+			(type default)
+		)
+	)
+	(wire
+		(pts
 			(xy 38.1 25.4) (xy 38.1 38.1)
 		)
@@
 	(wire
 		(pts
+			(xy 138.43 55.88) (xy 144.78 55.88)
+		)
+		(stroke
+			(width 0)
+			(type default)
+		)
+	)
+	(wire
+		(pts
 			(xy 38.1 50.8) (xy 38.1 63.5)
 		)
@@
 		(pts
 			(xy 60.96 71.12) (xy 73.66 71.12)
+		)
+		(stroke
+			(width 0)
+			(type default)
+		)
+	)
+	(wire
+		(pts
+			(xy 160.02 31.75) (xy 160.02 34.29)
 		)
 		(stroke
@@
 	)
 	(label "COL0"
-		(at 110.49 44.45 180)
+		(at 144.78 48.26 180)
 		(effects
 			(font
@@
 	)
 	(label "COL2"
-		(at 110.49 49.53 180)
+		(at 144.78 53.34 180)
 		(effects
 			(font
@@
 	)
 	(label "ROW0"
-		(at 110.49 36.83 180)
+		(at 144.78 40.64 180)
 		(effects
 			(font
@@
 	)
 	(label "ROW1"
-		(at 110.49 39.37 180)
+		(at 144.78 43.18 180)
 		(effects
 			(font
@@
 	)
 	(label "COL1"
-		(at 110.49 46.99 180)
+		(at 144.78 50.8 180)
 		(effects
 			(font
@@
 	)
 	(label "ROW2"
-		(at 110.49 41.91 180)
+		(at 144.78 45.72 180)
 		(effects
 			(font
@@
 	)
 	(symbol
+		(lib_id "Connector_Audio:AudioPlug4")
+		(at 116.84 59.69 0)
+		(unit 1)
+		(body_style 1)
+		(exclude_from_sim no)
+		(in_bom yes)
+		(on_board yes)
+		(in_pos_files yes)
+		(dnp no)
+		(fields_autoplaced yes)
+		(property "Reference" "J1"
+			(at 116.84 50.8 0)
+			(show_name no)
+			(do_not_autoplace no)
+			(effects
+				(font
+					(size 1.27 1.27)
+				)
+			)
+		)
+		(property "Value" "AudioPlug4"
+			(at 116.84 53.34 0)
+			(show_name no)
+			(do_not_autoplace no)
+			(effects
+				(font
+					(size 1.27 1.27)
+				)
+			)
+		)
+		(property "Footprint" ""
+			(at 125.73 62.23 0)
+			(hide yes)
+			(show_name no)
+			(do_not_autoplace no)
+			(effects
+				(font
+					(size 1.27 1.27)
+				)
+			)
+		)
+		(property "Datasheet" ""
+			(at 125.73 62.23 0)
+			(hide yes)
+			(show_name no)
+			(do_not_autoplace no)
+			(effects
+				(font
+					(size 1.27 1.27)
+				)
+			)
+		)
+		(property "Description" "Audio Jack, 4 Poles (Stereo / TRRS)"
+			(at 116.84 59.69 0)
+			(hide yes)
+			(show_name no)
+			(do_not_autoplace no)
+			(effects
+				(font
+					(size 1.27 1.27)
+				)
+			)
+		)
+		(pin "R2"
+		)
+		(pin "R1"
+		)
+		(pin "T"
+		)
+		(pin "S"
+		)
+		(instances
+			(project "macro9000"
+				(path "/25bc4964-606a-46d2-b40e-61fd1c96fe32"
+					(reference "J1")
+					(unit 1)
+				)
+			)
+		)
+	)
+	(symbol
 		(lib_id "Switch:SW_Push")
 		(at 55.88 50.8 0)
@@
 	(symbol
 		(lib_id "rp2040-zero:RP2040-Zero")
-		(at 124.46 46.99 0)
+		(at 158.75 50.8 0)
 		(unit 1)
 		(body_style 1)
@@
 		(fields_autoplaced yes)
 		(property "Reference" "RZ1"
-			(at 126.6033 64.77 0)
+			(at 160.8933 68.58 0)
 			(show_name no)
 			(do_not_autoplace no)
@@
 		)
 		(property "Value" "RP2040-Zero"
-			(at 126.6033 67.31 0)
+			(at 160.8933 71.12 0)
 			(show_name no)
 			(do_not_autoplace no)
@@
 		)
 		(property "Footprint" "MacroKeys:RP2040-Zero"
-			(at 126.6033 69.85 0)
+			(at 160.8933 73.66 0)
 			(show_name no)
 			(do_not_autoplace no)
@@
 		)
 		(property "Datasheet" ""
-			(at 124.46 46.99 0)
+			(at 158.75 50.8 0)
 			(hide yes)
 			(show_name no)
@@
 		)
 		(property "Description" ""
-			(at 124.46 46.99 0)
-			(hide yes)
-			(show_name no)
+			(at 158.75 50.8 0)
+			(hide yes)
+			(show_name no)
